File: EPC_val/EPC_val.kicad_pcb (KiCad board)
At the start: 4 copper layers, 74 x 43 mm, 37 parts, among them J1 691137710002, J2 691137710002, J3 691137710002, Q1 EPC2304ENGRT, Q2 EPC2304ENGRT, U1 NCP51820AMNTWG

Commit message: need to fix vias
Routing:
- net +12V: track 40.0 -> 41.5 mm
- net GND: vias 16 -> 22
Changed lines of the file:
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@@
+	)
+	(via
+		(at 167.125 103.975)
+		(size 0.6)
+		(drill 0.3)
+		(layers "F.Cu" "B.Cu")
+		(net 2)
 	)
 	(via
@@
 	)
 	(via
+		(at 167.125 102.975)
+		(size 0.6)
+		(drill 0.3)
+		(layers "F.Cu" "B.Cu")
+		(net 2)
+	)
+	(via
+		(at 167.125 101.975)
+		(size 0.6)
+		(drill 0.3)
+		(layers "F.Cu" "B.Cu")
+		(net 2)
+	)
+	(via
 		(at 163.225 106.75)
 		(size 0.6)
@@
 	)
 	(via
+		(at 177.017054 104.20404)
+		(size 0.6)
+		(drill 0.3)
+		(layers "F.Cu" "B.Cu")
+		(net 2)
+	)
+	(via
+		(at 177.375 104.975)
+		(size 0.6)
+		(drill 0.3)
+		(layers "F.Cu" "B.Cu")
+		(net 2)
+	)
+	(via
 		(at 170.825 102)
 		(size 0.6)
@@
 		(layers "F.Cu" "B.Cu")
 		(free yes)
+		(net 2)
+	)
+	(via
+		(at 176.4 104.975)
+		(size 0.6)
+		(drill 0.3)
+		(layers "F.Cu" "B.Cu")
 		(net 2)
 	)
@@
 	)
 	(segment
-		(start 165.4 117.175)
-		(end 183.725 98.85)
-		(width 0.5)
-		(layer "B.Cu")
-		(net 9)
-	)
-	(segment
-		(start 161.175 117.175)
-		(end 165.4 117.175)
-		(width 0.5)
-		(layer "B.Cu")
-		(net 9)
-	)
-	(segment
-		(start 183.725 98.85)
+		(start 178.8 103.725)
 		(end 183.725 98.8)
 		(width 0.5)
@@
 	)
 	(segment
+		(start 161.175 117.175)
+		(end 167.9 117.175)
+		(width 0.5)
+		(layer "B.Cu")
+		(net 9)
+	)
+	(segment
 		(start 159 115)
 		(end 161.175 117.175)
+		(width 0.5)
+		(layer "B.Cu")
+		(net 9)
+	)
+	(segment
+		(start 167.9 117.175)
+		(end 178.8 106.275)
+		(width 0.5)
+		(layer "B.Cu")
+		(net 9)
+	)
+	(segment
+		(start 178.8 106.275)
+		(end 178.8 103.725)
 		(width 0.5)
 		(layer "B.Cu")
@@
 		(polygon
 			(pts
-				(xy 181 79) (xy 187 79) (xy 187 86) (xy 193 86) (xy 193 92) (xy 181 92)
+				(xy 181 78) (xy 187 78) (xy 187 86) (xy 193 86) (xy 193 92) (xy 181 92)
 			)
 		)
@@
 		(polygon
 			(pts
-				(xy 167.525 96.325) (xy 152 96.325) (xy 152 102.5) (xy 167.525 102.5)
+				(xy 165.35 102.5) (xy 167.525 100.775) (xy 167.525 96.325) (xy 152 96.325) (xy 152 102.5)
 			)
 		)
@@
 		(polygon
 			(pts
-				(xy 168 79) (xy 177 79) (xy 177 92) (xy 165 92) (xy 165 94) (xy 162 94) (xy 161.2 94.8) (xy 161.2 96.325)
+				(xy 169.041968 78) (xy 177 78) (xy 177 92) (xy 165 92) (xy 165 94) (xy 162 94) (xy 161.2 94.8) (xy 161.2 96.325)
 				(xy 159.05 96.325) (xy 159 96.275) (xy 159 87.6375)
 			)
@@
 		(layer "F.Cu")
 		(hatch edge 0.5)
+		(priority 1)
 		(connect_pads yes
 			(clearance 1)
@@
 		(polygon
 			(pts
-				(xy 161.675 105.475) (xy 164.9 105.475) (xy 165.675 106.25) (xy 165.675 108) (xy 165.575 108.1)
-				(xy 160.675 108.1) (xy 160.675 106.475)
+				(xy 161.675 105.475) (xy 165 105.45) (xy 165.675 106.25) (xy 165.675 108) (xy 165.575 108.1) (xy 160.675 108.1)
+				(xy 160.675 106.475)
+			)
+		)
+	)
+	(zone
+		(net 6)
+		(net_name "/SW")
+		(layer "F.Cu")
+		(hatch edge 0.5)
+		(priority 3)
+		(connect_pads yes
+			(clearance 0.5)
+		)
+		(min_thickness 0.25)
+		(filled_areas_thickness no)
+		(fill yes
+			(thermal_gap 0.5)
+			(thermal_bridge_width 0.5)
+			(smoothing chamfer)
+			(radius 1)
+		)
+		(polygon
+			(pts
+				(xy 165.15 95.275) (xy 166.1 95.275) (xy 166.425 95.6) (xy 167.3 95.6) (xy 167.525 95.375) (xy 167.525 92.525)
+				(xy 167.3 92.3) (xy 165.9 92.3) (xy 165.15 93.05)
 			)
 		)
@@
 		(polygon
 			(pts
-				(xy 167 100.6) (xy 176.4 100.6) (xy 181 96) (xy 177 92) (xy 167 92)
+				(xy 181 96) (xy 176.4 100.6) (xy 167 100.6) (xy 167 92) (xy 177 92)
 			)
 		)
@@
 		(net 2)
 		(net_name "GND")
-		(layers "F.Cu" "In1.Cu" "In2.Cu" "B.Cu")
-		(hatch edge 0.5)
-		(connect_pads yes
-			(clearance 1)
+		(layers "F.Cu" "In1.Cu")
+		(hatch edge 0.5)
+		(priority 9)
+		(connect_pads yes
+			(clearance 0.2)
 		)
 		(min_thickness 0.25)
@@
 		(polygon
 			(pts
-				(xy 122 77) (xy 196 77) (xy 196 120) (xy 122 120)
+				(xy 165.35 102.5) (xy 167.1 100.75) (xy 176.4 100.75) (xy 178.6 102.95) (xy 178.6 104.525) (xy 175.8 107.325)
+				(xy 168.025 107.325) (xy 165.35 104.65)
+			)
+		)
+	)
+	(zone
+		(net 2)
+		(net_name "GND")
+		(layers "F.Cu" "In1.Cu" "In2.Cu" "B.Cu")
+		(hatch edge 0.5)
+		(connect_pads yes
+			(clearance 1)
+		)
+		(min_thickness 0.25)
+		(filled_areas_thickness no)
+		(fill yes
+			(thermal_gap 0.5)
+			(thermal_bridge_width 0.5)
+			(smoothing chamfer)
+			(radius 0.2)
+		)
+		(polygon
+			(pts
+				(xy 122 77) (xy 122 120) (xy 152 120) (xy 152 110) (xy 167.525 110) (xy 167.525 107) (xy 167.525 101.5)
+				(xy 165 101.5) (xy 165 93) (xy 167 91) (xy 196 91) (xy 196 77)
+			)
+		)
+	)
+	(zone
+		(net 2)
+		(net_name "GND")
+		(layers "F.Cu" "In1.Cu" "In2.Cu" "B.Cu")
+		(hatch edge 0.5)
+		(connect_pads yes
+			(clearance 1)
+		)
+		(min_thickness 0.25)
+		(filled_areas_thickness no)
+		(fill yes
+			(thermal_gap 0.5)
+			(thermal_bridge_width 0.5)
+			(smoothing chamfer)
+			(radius 1)
+		)
+		(polygon
+			(pts
+				(xy 155 120) (xy 155 111) (xy 168 111) (xy 168 107.35) (xy 168.025 107.325) (xy 175.8 107.325) (xy 182 101.125)
+				(xy 182 100) (xy 180 98) (xy 182 96) (xy 180 94) (xy 180 93) (xy 196 93) (xy 196 120)
 			)
 		)
@@
 		(layer "B.Cu")
 		(hatch edge 0.5)
-		(priority 6)
+		(priority 11)
 		(connect_pads yes
 			(clearance 0.5)

Commit message: epc board should be ready to order
Parts:
- added G***: LOGO, LOGO, F.Cu at (126.8, 82.0)
- added G***: LOGO, LOGO, F.Cu at (192.9, 96.5)
- added G***: LOGO, LOGO, F.Cu at (160.9, 99.5)
- renumbered J1 to 12V/GND, TP4 to GND, TP3 to GND, TP11 to GND, J2 to GND/L, Q1 to HS, TP1 to HS, J3 to HSD/GND, TP9 to HSG, Q2 to LS, TP2 to LS, TP10 to LSG, TP13 to SW
Routing:
- net GND: track 9.62 -> 10.8 mm, vias 22 -> 81
- net +12V: track 41.5 -> 42.6 mm
- net /SW: vias 20 -> 22
Other:
- board size 74 x 43 mm -> 75.6 x 43 mm
- board text added: "EPC Dev Board"
- board text added: "Rev 1.0 April 2024"
