File: HEI_Power_Stage/Power_Stage/Power_Stage/isolation.kicad_sch (KiCad schematic)
At the start: 7 parts, among them U1 TBA 2-1212, U18 ISO6741, U19 ISO6741

Commit message: more isolation
Parts:
- added U20: ISO6760, SOIC16_ISO6760_DW_TEX, symbol ISO6760:XISO6760FDWR
Connections:
- net +3V3_LV: now also U20.1 (VCC1)
- net +5V: now also U20.16 (VCC2); no longer U18.10 (EN2), U18.16 (V_{CC2}), U19.10 (EN2), U19.16 (V_{CC2})
- net GND: now also U20.9 (GND2)
- net GND_LV: now also U20.8 (GND1)
- new net +5V_HV: U18.10 (EN2), U18.16 (V_{CC2}), U19.10 (EN2), U19.16 (V_{CC2})
- new net AH: U20.15 (OUTA)
- new net AH_LV: U20.2 (INA)
- new net AL: U20.14 (OUTB)
- new net AL_LV: U20.3 (INB)
- new net BH: U20.13 (OUTC)
- new net BH_LV: U20.4 (INC)
- new net BL: U20.12 (OUTD)
- new net BL_LV: U20.5 (IND)
- new net CH: U20.11 (OUTE)
- new net CH_LV: U20.6 (INE)
- new net CL: U20.10 (OUTF)
- new net CL_LV: U20.7 (INF)
Other:
- note added: "PWM Isolator (GND ref)"
- note added: "SPI Isolator (HV- ref)"
- note removed: "SPI Isolator"

Commit message: small changes
Parts:
- added TP1, TP2, TP3, TP4: Test_Point, TestPoint:TestPoint_Keystone_5000-5004_Miniature, symbol GTSR_Libraries:Test_Point
- U1: footprint GTSR_KiCAD_Footprints_SD:TBA 2_SINGLE_TRP -> GTSR:TBA 2_SINGLE_TRP
Connections:
- net +12V_LV: now also TP1.1
- net GND_LV: now also TP3.1
Other:
- note added: "Needs to cross HV gap"
- note removed: "Add more testpoints"
