File: HEI_Power_Stage/Power_Stage/Power_Stage/Power_Stage.kicad_pcb (KiCad board)
At the start: 4 copper layers, 114.7 x 57.4 mm, 175 parts, among them J1 Screw_Terminal_01x01, J2 Conn_02x10_Odd_Even, J3 Screw_Terminal_01x01, J4 Screw_Terminal_01x01, J5 Screw_Terminal_01x01, J6 Screw_Terminal_01x01, Q1 EPC2304ENGRT, Q2 EPC2304ENGRT, Q3 EPC2304ENGRT, Q4 EPC2304ENGRT, Q5 EPC2304ENGRT, Q6 EPC2304ENGRT, T1 30k, T2 30k, T3 30k, T4 30k, T5 30k, T6 30k, U1 TBA 2-1212, U11 NCP51820AMNTWG, U12 ADC124S051CIMM/NOPB, U13 TPS73250DBVR, U14 TPS73250DBVR, U15 ADC124S051CIMM/NOPB, U17 TPS73250DBVR, U18 ISO6741, U19 ISO6741, U2 1769205241, U20 ISO6760, U21 1769205241, U3 TPS73250DBVR, U5 NCP51820AMNTWG, U6 ADC124S051CIMM/NOPB, U8 NCP51820AMNTWG, U9 ADC124S051CIMM/NOPB

Commit message: I think all schematic done
added new mps gate driver, new acs current sense, new differential voltage sense, new 5-5 iso converters.
beginning layout
Parts:
- removed C10, C22, C6, C7, C8: 10uF, Capacitor_SMD:C_0603_1608Metric_Pad1.08x0.95mm_HandSolder
- removed C13, C25: 1nF, Capacitor_SMD:C_0603_1608Metric_Pad1.08x0.95mm_HandSolder
- removed C19, C31: 0.1uF, Capacitor_SMD:C_0603_1608Metric_Pad1.08x0.95mm_HandSolder
- removed C20, C32: 1uF, Capacitor_SMD:C_0603_1608Metric_Pad1.08x0.95mm_HandSolder
- removed the C4 at (174.3, 112.4)
- removed the C4 at (169.0, 63.1)
- removed the C5 at (169.0, 65.6)
- removed the C5 at (165.3, 112.3)
- removed the D1 at (164.7, 80.5)
- removed the D1 at (158.3, 111.4)
- removed JP1, JP2, JP3: Jumper_2_Open, Jumper:SolderJumper-2_P1.3mm_Open_RoundedPad1.0x1.5mm
- removed the R1 at (161.3, 112.3)
- removed the R1 at (169.0, 68.1)
- removed R17, R37: 715k, Resistor_SMD:R_1206_3216Metric
- removed R31, R38: 10k, Resistor_SMD:R_1206_3216Metric
- removed R33, R5: 2.2 0.1W, Resistor_SMD:R_0603_1608Metric_Pad0.98x0.95mm_HandSolder
- removed R34, R6: 50k, Resistor_SMD:R_0603_1608Metric_Pad0.98x0.95mm_HandSolder
- removed R35, R39: 10k, Resistor_SMD:R_0603_1608Metric_Pad0.98x0.95mm_HandSolder
- removed R36: 2 1/16W, Resistor_SMD:R_0603_1608Metric_Pad0.98x0.95mm_HandSolder
- removed R41, R43: 0 1/16W, Resistor_SMD:R_0603_1608Metric_Pad0.98x0.95mm_HandSolder
- removed R45, R46, R47, R48, R49, R50, R51, R57: 2.2 0.1W, Resistor_SMD:R_0402_1005Metric_Pad0.72x0.64mm_HandSolder
- removed T1, T2, T3, T4, T5, T6: 30k, GTSR_KiCAD_Footprints_SD:2152723803
- removed TP1, TP11, TP12, TP2, TP3, TP4: Test_Point, TestPoint:TestPoint_Keystone_5000-5004_Miniature
- removed U1: TBA 2-1212, GTSR:TBA 2_SINGLE_TRP
- removed U10, U4, U7: ~, GTSR_KiCAD_Footprints_SD:XDCR_ACS72981LLRATR-100B5
- removed U11, U8: NCP51820AMNTWG, GTSR_KiCAD_Footprints:QFN_0AMNTWG_ONS-L
- removed U12, U6, U9: ADC124S051CIMM/NOPB, GTSR_KiCAD_Footprints:SOP50P490X110-10N
- removed U13, U14, U17: TPS73250DBVR, Package_TO_SOT_SMD:TSOT-23-5
- removed U15: ADC124S051CIMM/NOPB, GTSR:SOP50P490X110-10N
- removed U16: ~, GTSR:XDCR_ACS72981LLRATR-100B5
- removed U18, U19: ISO6741, Package_SO:SOIC-16W_7.5x10.3mm_P1.27mm
- removed U20: ISO6760, iso6760:SOIC16_ISO6760_DW_TEX
- removed U21: 1769205241, GTSR:176920512
- added C4: B58035U5106M001, B58035U5106M001_KiCad:B58035U5106M001, F.Cu at (92.2, 54.1)
- added C5: B58035U5106M001, B58035U5106M001_KiCad:B58035U5106M001, F.Cu at (106.0, 54.1)
- added C57: 4.7uF, Capacitor_SMD:C_0603_1608Metric_Pad1.08x0.95mm_HandSolder, F.Cu at (255.1, 78.0)
- added C58: 4.7uF, Capacitor_SMD:C_0603_1608Metric_Pad1.08x0.95mm_HandSolder, F.Cu at (183.2, 129.6)
- added C59: 1uF, Capacitor_SMD:C_0603_1608Metric_Pad1.08x0.95mm_HandSolder, F.Cu at (49.3, 162.7)
- added C60: 1uF, Capacitor_SMD:C_0603_1608Metric_Pad1.08x0.95mm_HandSolder, F.Cu at (247.6, 66.8)
- added C61: 1uF, Capacitor_SMD:C_0603_1608Metric_Pad1.08x0.95mm_HandSolder, F.Cu at (183.2, 132.2)
- added C62: 4.7uF, Capacitor_SMD:C_0603_1608Metric_Pad1.08x0.95mm_HandSolder, F.Cu at (49.3, 165.2)
- added C64: 4.7uF, Capacitor_SMD:C_0603_1608Metric_Pad1.08x0.95mm_HandSolder, F.Cu at (183.2, 134.7)
- added C65: 4.7uF, Capacitor_SMD:C_0603_1608Metric_Pad1.08x0.95mm_HandSolder, F.Cu at (94.4, 126.4)
- added C66: 1uF, Capacitor_SMD:C_0603_1608Metric_Pad1.08x0.95mm_HandSolder, F.Cu at (94.4, 128.9)
- added C67: 4.7uF, Capacitor_SMD:C_0603_1608Metric_Pad1.08x0.95mm_HandSolder, F.Cu at (98.7, 121.4)
- added D1: G, LED_SMD:LED_0603_1608Metric_Pad1.05x0.95mm_HandSolder, F.Cu at (108.7, 121.4)
- added D10: 5.1-5.7v, Diode_SMD:D_SOD-128, F.Cu at (142.4, 95.7)
- added D11: 5.1-5.7v, Diode_SMD:D_SOD-128, F.Cu at (190.8, 78.9)
- added D12: 5.1-5.7v, Diode_SMD:D_SOD-128, F.Cu at (201.9, 145.2)
- added D13: 5.1-5.7v, Diode_SMD:D_SOD-128, F.Cu at (64.6, 125.2)
- added D6: ~, Diode_SMD:D_SOD-523, F.Cu at (204.4, 148.4)
- added D7: G, LED_SMD:LED_0603_1608Metric_Pad1.05x0.95mm_HandSolder, F.Cu at (66.5, 179.0)
- added D8: G, LED_SMD:LED_0603_1608Metric_Pad1.05x0.95mm_HandSolder, F.Cu at (253.0, 80.2)
- added D9: G, LED_SMD:LED_0603_1608Metric_Pad1.05x0.95mm_HandSolder, F.Cu at (200.4, 148.5)
- added IC1: ACS730KLCTR-65ABT, ACS730KLCTR65ABT_KiCad:SOIC127P600X175-8N, F.Cu at (162.2, 92.1)
- added IC2: ACS730KLCTR-65ABT, ACS730KLCTR65ABT_KiCad:SOIC127P600X175-8N, F.Cu at (184.7, 93.8)
- added IC3: ACS730KLCTR-65ABT, ACS730KLCTR65ABT_KiCad:SOIC127P600X175-8N, F.Cu at (193.9, 146.4)
- added IC4: AMC1311DWVR, AMC1311_KiCad:SOIC127P1150X280-8N, F.Cu at (94.9, 116.4)
- added IC9: ACS730KLCTR-65ABT, ACS730KLCTR65ABT_KiCad:SOIC127P600X175-8N, F.Cu at (65.1, 119.9)
- added J7: Conn_02x10_Odd_Even, Connector_PinHeader_2.54mm:PinHeader_2x10_P2.54mm_Horizontal, F.Cu at (90.3, 87.5)
- added PS1: CRE1S0505MC, CRE1S0505MC_KiCad:CRE1S0505MC, F.Cu at (63.7, 158.8)
- added PS2: CRE1S0505MC, CRE1S0505MC_KiCad:CRE1S0505MC, F.Cu at (255.5, 69.4)
- added PS3: CRE1S0505MC, CRE1S0505MC_KiCad:CRE1S0505MC, F.Cu at (197.6, 128.3)
- added PS4: CRE1S0505MC, CRE1S0505MC_KiCad:CRE1S0505MC, F.Cu at (79.9, 120.0)
- added R1: 0, Resistor_SMD:R_0603_1608Metric_Pad0.98x0.95mm_HandSolder, F.Cu at (180.0, 65.8)
- added R77: 1.2k, Resistor_SMD:R_0603_1608Metric_Pad0.98x0.95mm_HandSolder, F.Cu at (98.7, 128.9)
- C1, C2, C3: footprint GTSR_KiCAD_Footprints:CAP_6050_TDK -> GTSR:CAP_6050_TDK
- C11: value 15pF -> 0.1uF
- C12, C23: value 15pF -> 1nF
- C15: value 1uF -> 1nF
- C16, C18: value 1uF -> 0.1uF
- C17: value 470nF -> 1nF
- C21, C9: value 0.1uF -> 10uF
- C24: value 15pF -> 10uF
- C26, C34, C43, C46: value 0.1uF -> 1uF
- C29: value 470nF -> 0.1uF
- C30: value 1uF -> 0.1uF; moved to B.Cu
- C35, C36: value 15pF -> 2.2nF
- C37: value 1nF -> 100nF
- C38: value 0.1uF -> 2.2nF
- C40, C45: moved to B.Cu
- C41: value 470nF -> 1uF
- C44: value 1uF -> 100nF
- C47: value 1nF -> 0.1uF
- C48: value 10uF -> 0.1uF; moved to B.Cu
- C49, C50: moved to F.Cu
- C51, C52: value 10uF -> 0.1uF
- C54: value 15pF -> 0.1uF; footprint Capacitor_SMD:C_0402_1005Metric_Pad0.74x0.62mm_HandSolder -> Capacitor_SMD:C_0603_1608Metric_Pad1.08x0.95mm_HandSolder; moved to B.Cu
- C55: value 15pF -> 0.1uF; footprint Capacitor_SMD:C_0402_1005Metric_Pad0.74x0.62mm_HandSolder -> Capacitor_SMD:C_0603_1608Metric_Pad1.08x0.95mm_HandSolder
- C56, C63: value 15pF -> 4.7uF; footprint Capacitor_SMD:C_0402_1005Metric_Pad0.74x0.62mm_HandSolder -> Capacitor_SMD:C_0603_1608Metric_Pad1.08x0.95mm_HandSolder
- D3: value RFU02VSM6STR -> G; footprint GTSR_KiCAD_Footprints:DIO_RFU02VS_ROM-M -> LED_SMD:LED_0603_1608Metric_Pad1.05x0.95mm_HandSolder
- D4, D5: value RFU02VSM6STR -> ~; footprint GTSR_KiCAD_Footprints:DIO_RFU02VS_ROM-M -> Diode_SMD:D_SOD-523
- J3, J4, J5: footprint GTSR_KiCAD_Footprints_SD:CONN6_1057_WRE -> GTSR:CONN6_1057_WRE
- Q1, Q2, Q3, Q4, Q5, Q6: footprint GTSR_KiCAD_Footprints:EPC2304_ECC -> GTSR:EPC2304_ECC; moved to B.Cu
- R10: value 10k -> 0; footprint Resistor_SMD:R_1206_3216Metric -> Resistor_SMD:R_0603_1608Metric_Pad0.98x0.95mm_HandSolder
- R11, R7: value 10k -> 0
- R12, R14, R26, R28, R40, R42: value 0.47 1/16W -> 10
- R13, R15: value 0 1/16W -> 0
- R16: value 330 -> 1Meg; footprint Resistor_SMD:R_0603_1608Metric_Pad0.98x0.95mm_HandSolder -> Resistor_SMD:R_1206_3216Metric
- R18, R4: value 2.2 0.1W -> 0
- R19: value 2.2 0.1W -> 10k
- R20: value 50k -> 10k
- R22, R8: value 2 1/16W -> 0
- R23: value 715k -> 0; footprint Resistor_SMD:R_1206_3216Metric -> LED_SMD:LED_0603_1608Metric_Pad1.05x0.95mm_HandSolder
- R24: value 10k -> 0; footprint Resistor_SMD:R_1206_3216Metric -> LED_SMD:LED_0603_1608Metric_Pad1.05x0.95mm_HandSolder
- R25: value 10k -> 0; footprint Resistor_SMD:R_0603_1608Metric_Pad0.98x0.95mm_HandSolder -> LED_SMD:LED_0603_1608Metric_Pad1.05x0.95mm_HandSolder
- R27, R29: value 0 1/16W -> 440
- R3: value 330 -> 0
- R30: value 330 -> 10k; footprint Resistor_SMD:R_0603_1608Metric_Pad0.98x0.95mm_HandSolder -> Resistor_SMD:R_1206_3216Metric
- R32: value 2.2 0.1W -> 440
- R44: value 330 -> 440
- R9: value 715k -> 0; footprint Resistor_SMD:R_1206_3216Metric -> Resistor_SMD:R_0603_1608Metric_Pad0.98x0.95mm_HandSolder
- U2: value 1769205241 -> MP18831-4AGY; footprint GTSR_KiCAD_Footprints_SD:176920512 -> Package_SO:SOIC-16W_7.5x10.3mm_P1.27mm
- U3: value TPS73250DBVR -> MP18831-4AGY; footprint Package_TO_SOT_SMD:TSOT-23-5 -> Package_SO:SOIC-16W_7.5x10.3mm_P1.27mm
- U5: value NCP51820AMNTWG -> MP18831-4AGY; footprint GTSR_KiCAD_Footprints:QFN_0AMNTWG_ONS-L -> Package_SO:SOIC-16W_7.5x10.3mm_P1.27mm
- moved C63 154.4 mm to (245.8, 66.8), turned to -90 degrees
- moved C56 131.7 mm to (49.3, 160.2), turned to 0 degrees
- moved J5 126.1 mm to (55.4, 88.2), turned to 0 degrees
- moved R29 118.7 mm to (256.7, 80.3), turned to 0 degrees
- moved J4 112.4 mm to (45.6, 88.2), turned to 0 degrees
- moved J3 100.4 mm to (35.8, 88.2), turned to 0 degrees
- moved C3 98.3 mm to (65.9, 113.0)
- moved R11 97.4 mm to (186.9, 65.9), turned to -90 degrees
- moved H3 96.2 mm to (106.8, 99.5)
- moved C45 96.1 mm to (178.2, 81.5), turned to 0 degrees
- moved C48 95.5 mm to (184.7, 79.8), turned to 0 degrees
- moved C46 93.5 mm to (183.2, 122.1), turned to 0 degrees
- moved R8 93.0 mm to (185.3, 65.8), turned to -90 degrees
- moved R27 91.9 mm to (53.6, 162.7), turned to 0 degrees
- moved U3 91.4 mm to (181.5, 74.3), turned to -90 degrees
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Connections:
- C11 pad 1: /Phase1/HIN -> +5V_LV
- C12 pad 1: /Phase1/LIN -> /DCI_{sense}ref
- C14 pad 1: GND -> +5V_LV
- C14 pad 2: /Phase1/DT -> GND
- C15 pad 1: /Phase1/VDDH -> /PHAI_{sense}ref
- C15 pad 2: /Phase1/SW -> GND
- C16 pad 1: HV- -> +5V_LV
- C16 pad 2: /Phase1/VDDL -> GND
- C17 pad 1: /Phase1/V_{BST} -> /PHBI_{sense}ref
- C17 pad 2: /Phase1/SW -> GND
- C18 pad 1: +12V -> +5V_LV
- C21 pad 1: /5VrefB -> GND
- C21 pad 2: HV- -> +5V_LV
- C23 pad 1: /Phase2/HIN -> /PHCI_{sense}ref
- C24 pad 1: /Phase2/LIN -> GND
- C24 pad 2: GND -> +5V_LV
- C26 pad 2: /Phase2/DT -> +5V_LV
- C27 pad 1: /Phase2/VDDH -> GND
- C27 pad 2: /Phase2/SW -> +5V_LV
- C28 pad 1: HV- -> GND
- C28 pad 2: /Phase2/VDDL -> +5V_LV
- C29 pad 1: /Phase2/V_{BST} -> GND
- C29 pad 2: /Phase2/SW -> +5V_LV
- C30 pad 1: +12V -> GND
- C30 pad 2: GND -> +5V_LV
- C33 pad 1: /5VrefC -> GND
- C33 pad 2: HV- -> +5V_LV
- C34 pad 1: /5VrefDC -> HV-
- C34 pad 2: HV- -> +5V_HV
- C35 pad 1: /Phase3/HIN -> GND
- C35 pad 2: GND -> /Phase1/DT
- C36 pad 1: /Phase3/LIN -> GND
- C36 pad 2: GND -> /Phase2/DT
- C37 pad 1: /Phase3/I_{ADC} -> HV-
- C37 pad 2: HV- -> +5V_HV
- C39 pad 1: /Phase3/VDDH -> /Phase1/SW
- C39 pad 2: /Phase3/SW -> /Phase1/VDDhs
- C40 pad 1: HV- -> /Phase2/SW
- C40 pad 2: /Phase3/VDDL -> /Phase2/VDDhs
- C41 pad 1: /Phase3/V_{BST} -> /Phase3/SW
- C41 pad 2: /Phase3/SW -> /Phase3/VDDhs
- C42 pad 1: +12V -> HV-
- C42 pad 2: GND -> +5V_HV
- C43 pad 1: /5VrefC -> GND
- C43 pad 2: HV- -> +5V_LV
- C44 pad 1: /5VrefC -> GND
- C44 pad 2: HV- -> +5V_LV
- C45 pad 1: /5VrefDC -> HV-
- C45 pad 2: HV- -> +5V_HV
- C46 pad 1: /5VrefDC -> HV-
- C46 pad 2: HV- -> +5V_HV
- C47 pad 1: /I_{DC} -> /Phase1/SW
- C47 pad 2: HV- -> /Phase1/VDDhs
- C48 pad 1: +5V_HV -> /Phase2/SW
- C48 pad 2: HV- -> /Phase2/VDDhs
- C51 pad 1: +12V -> /Phase3/SW
- C51 pad 2: GND -> /Phase3/VDDhs
- C52 pad 1: +5V -> HV-
- C52 pad 2: GND -> +5V_HV
- C54 pad 1: /Phase1/V_{ADC} -> HV-
- C54 pad 2: HV- -> +5V_HV
- C55 pad 1: /Phase2/V_{ADC} -> HV-
- C55 pad 2: HV- -> +5V_HV
- C56 pad 1: /Phase3/V_{ADC} -> /Phase1/SW
- C56 pad 2: HV- -> /Phase1/VDDA
- C63 pad 1: /V_{DC} -> GND
- C63 pad 2: HV- -> +5V_LV
- C9 pad 1: /5VrefA -> GND
- C9 pad 2: HV- -> +5V_LV
- D2 pad 1: HV- -> GND
- D3 pad 1: Net-(D3-K) -> GND
- D3 pad 2: +12V -> Net-(D3-A)
- D4 pad 1: Net-(D4-K) -> /Phase1/VDDhs
- D4 pad 2: +12V -> Net-(D4-A)
- D5 pad 1: Net-(D5-K) -> /Phase2/VDDhs
- D5 pad 2: +12V -> Net-(D5-A)
- J2 pad 10: /MOSI_LV -> unconnected-(J2-Pin_10-Pad10)
- J2 pad 12: /MISO_LV -> unconnected-(J2-Pin_12-Pad12)
- J2 pad 14: /CLK_LV -> unconnected-(J2-Pin_14-Pad14)
- J2 pad 18: +3V3_LV -> unconnected-(J2-Pin_18-Pad18)
- J2 pad 19: /12V_LV -> +12V_LV
- J2 pad 2: /DC~{CS}_LV -> unconnected-(J2-Pin_2-Pad2)
- J2 pad 20: /GND_LV -> GND
- J2 pad 4: /C~{CS}_LV -> unconnected-(J2-Pin_4-Pad4)
- J2 pad 6: /B~{CS}_LV -> unconnected-(J2-Pin_6-Pad6)
- J2 pad 8: /A~{CS}_LV -> unconnected-(J2-Pin_8-Pad8)
- R10 pad 1: HV- -> /AHS_{PWM}
- R10 pad 2: /Phase1/V_{sense} -> /Phase1/INA
- R11 pad 1: /5VrefA -> /BHS_{PWM}
- R11 pad 2: /Phase1/LS_{Tsense} -> /Phase2/INA
- R12 pad 1: /Phase1/HS_{SRC} -> /Phase1/HS_{DRV}
- R13 pad 1: /Phase1/HS_{SNK} -> /Phase1/VDDA
- R13 pad 2: /Phase1/HS_{Gate} -> /Phase1/VDDhs
- R14 pad 1: /Phase1/LS_{SRC} -> /Phase1/LS_{DRV}
- R15 pad 1: /Phase1/LS_{SNK} -> /Phase2/VDDA
- R15 pad 2: /Phase1/LS_{Gate} -> /Phase2/VDDhs
- R16 pad 1: Net-(U6-DOUT) -> Net-(IC4-VIN)
- R16 pad 2: /MISO -> HV+
- R18 pad 1: /Phase2/HIN -> /CHS_{PWM}
- R18 pad 2: /BHS_{PWM} -> /Phase3/INA
- R19 pad 1: /Phase2/LIN -> /Phase1/DT
- R19 pad 2: /BLS_{PWM} -> GND
- R2 pad 2: +5V_HV -> +5V_LV
- R20 pad 1: GND -> /Phase2/DT
- R20 pad 2: /Phase2/DT -> GND
- R21 pad 1: /5VrefB -> /Phase3/DT
- R21 pad 2: /Phase2/HS_{Tsense} -> GND
- R22 pad 1: Net-(D4-K) -> /Phase3/VDDA
- R22 pad 2: /Phase2/V_{BST} -> /Phase3/VDDhs
- R23 pad 1: /Phase2/V_{sense} -> Net-(D4-A)
- R23 pad 2: /PHB -> +5V_HV
- R24 pad 1: HV- -> Net-(D5-A)
- R24 pad 2: /Phase2/V_{sense} -> +5V_HV
- R25 pad 1: /5VrefB -> Net-(D6-A)
- R25 pad 2: /Phase2/LS_{Tsense} -> +5V_HV
- R26 pad 1: /Phase2/HS_{SRC} -> /Phase2/HS_{DRV}
- R27 pad 1: /Phase2/HS_{SNK} -> Net-(D7-A)
- R27 pad 2: /Phase2/HS_{Gate} -> /Phase1/VDDA
- R28 pad 1: /Phase2/LS_{SRC} -> /Phase2/LS_{DRV}
- R29 pad 1: /Phase2/LS_{SNK} -> Net-(D8-A)
- R29 pad 2: /Phase2/LS_{Gate} -> /Phase2/VDDA
- R3 pad 1: Net-(U15-DOUT) -> +5V_LV
- R3 pad 2: /MOSI -> /Phase1/EN
- R30 pad 1: Net-(U9-DOUT) -> HV-
- R30 pad 2: /MISO -> Net-(IC4-VIN)
- R32 pad 1: /Phase3/HIN -> Net-(D9-A)
- R32 pad 2: /CHS_{PWM} -> /Phase3/VDDA
- R4 pad 1: /Phase1/HIN -> +5V_LV
- R4 pad 2: /AHS_{PWM} -> /Phase3/EN
- R40 pad 1: /Phase3/HS_{SRC} -> /Phase3/HS_{DRV}
- R42 pad 1: /Phase3/LS_{SRC} -> /Phase3/LS_{DRV}
- R44 pad 2: /MISO -> +5V_HV
- R7 pad 1: /5VrefA -> /ALS_{PWM}
- R7 pad 2: /Phase1/HS_{Tsense} -> /Phase1/INB
- R8 pad 1: Net-(D3-K) -> /BLS_{PWM}
- R8 pad 2: /Phase1/V_{BST} -> /Phase2/INB
- R9 pad 1: /Phase1/V_{sense} -> /CLS_{PWM}
- R9 pad 2: /PHA -> /Phase3/INB
- U2 pad 1: GND -> /Phase1/INA
- U2 pad 2: +12V -> /Phase1/INB
- U2 pad 4: HV- -> GND
- U2 pad 5: +5V_HV -> /Phase1/EN
- U2 pad 8: unconnected-(U2-NC-Pad8) -> +5V_LV
- U3 pad 1: +5V_HV -> /Phase2/INA
- U3 pad 2: HV- -> /Phase2/INB
- U3 pad 3: +5V_HV -> +5V_LV
- U3 pad 4: unconnected-(U3-NC-Pad4) -> GND
- U3 pad 5: /5VrefA -> /Phase2/EN
- U5 pad 1: /Phase1/VDDH -> /Phase3/INA
- U5 pad 10: GND -> /Phase3/LS_{DRV}
- U5 pad 11: /Phase1/LIN -> +5V_HV
- U5 pad 12: /Phase1/HIN -> unconnected-(U5-NC-Pad12)
- U5 pad 13: +12V -> unconnected-(U5-NC-Pad13)
- U5 pad 14: +12V -> /Phase3/SW
- U5 pad 15: /Phase1/V_{BST} -> /Phase3/HS_{DRV}
- U5 pad 2: /Phase1/HS_{SRC} -> /Phase3/INB
- U5 pad 3: /Phase1/HS_{SNK} -> +5V_LV
- U5 pad 4: /Phase1/SW -> GND
- U5 pad 5: /Phase1/VDDL -> /Phase3/EN
- U5 pad 6: /Phase1/LS_{SRC} -> /Phase3/DT
- U5 pad 7: /Phase1/LS_{SNK} -> unconnected-(U5-NC-Pad7)
- U5 pad 8: HV- -> +5V_LV
- U5 pad 9: /Phase1/DT -> HV-
Routing:
- net +5V: track 200.3 -> 0.00 mm, vias 4 -> 0
- net /CLK: track 181.5 -> 0.00 mm, vias 6 -> 0
- net /MOSI: track 172.6 -> 0.00 mm, vias 7 -> 0
- net /MISO: track 167.3 -> 0.00 mm, vias 7 -> 0
- net +12V: track 103.6 -> 0.00 mm, vias 4 -> 0
- net /C~{CS}: track 88.7 -> 0.00 mm, vias 2 -> 0
- net /B~{CS}: track 59.0 -> 0.00 mm, vias 2 -> 0
- net /GND_LV: track 56.3 -> 0.00 mm, vias 1 -> 0
- net +12V_LV: track 47.5 -> 0.00 mm
- net /A~{CS}: track 45.1 -> 0.00 mm, vias 1 -> 0
- net HV-: track 42.3 -> 0.00 mm, vias 188 -> 0
- net /CLS_{PWM}: track 42.1 -> 0.00 mm
- net /DC~{CS}: track 40.5 -> 0.00 mm, vias 2 -> 0
- net /CHS_{PWM}: track 37.7 -> 0.00 mm
- net GND: track 30.8 -> 0.00 mm, vias 42 -> 0
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- removed copper zone on B.Cu, net +3V3_LV
- removed copper zone on F.Cu, net /12V_LV
- removed copper zone on In1.Cu, net /GND_LV
- removed copper zone on F.Cu, net /PHA
- removed copper zone on In1.Cu, net /PHA
- removed copper zone on F.Cu, net /PHB
- removed copper zone on In1.Cu, net /PHB
- removed copper zone on F.Cu, net /PHC
- removed copper zone on In1.Cu, net /PHC
- removed copper zone on F.Cu, net /Phase1/SW
- removed copper zone on In1.Cu, net /Phase1/SW
- removed copper zone on F.Cu, net /Phase2/SW
- removed copper zone on In1.Cu, net /Phase2/SW
- removed copper zone on F.Cu, net /Phase3/SW
- removed copper zone on In1.Cu, net /Phase3/SW
- removed copper zone on F.Cu, net GND
- removed copper zone on In1.Cu, net GND
- removed copper zone on B.Cu, net HV+
- removed copper zone on F.Cu, net HV+
- removed copper zone on B.Cu, net HV+in
- removed copper zone on F.Cu, net HV+in
- removed copper zone on F.Cu, net HV-
- removed copper zone on In1.Cu, net HV-
- removed copper zone on In2.Cu, net HV-
Other:
- board outline removed
- board text removed: "Fill Pours Top half: gnd gnd pwrgnd pwrgnd -------- Bottom half: pwrgnd pwrgnd pwrgnd vdc Layer 3 gndpwr is full board"

Commit message: more progress
started placement for each half bridge
3d bodies
connectors sorted
options for dc link cap
Parts:
- removed C49: 210uF, kemet_cap:C4AQLEW6210A3BK
- removed J2, J7: Conn_02x10_Odd_Even, Connector_PinHeader_2.54mm:PinHeader_2x10_P2.54mm_Horizontal
- added C6: 15uF, C4AQLLU5150A19K _KiCad:C4AQLLU5150A19K, F.Cu at (43.2, 61.5)
- added J8: Conn_02x07_Odd_Even, Connector_PinSocket_2.54mm:PinSocket_2x07_P2.54mm_Vertical, F.Cu at (179.0, 42.2)
- added J9: Conn_02x07_Odd_Even, Connector_PinSocket_2.54mm:PinSocket_2x07_P2.54mm_Vertical, F.Cu at (131.4, 57.5)
- C29, C33, C39, C41, C42, C46, C47, C51, C52, C55: moved to B.Cu
- R12, R14, R26, R28, R40, R42: value 10 -> 0.75
- moved C56 214.1 mm to (254.9, 100.4)
- moved R27 211.9 mm to (256.8, 102.4)
- moved C59 210.8 mm to (246.8, 89.1), turned to -90 degrees
- moved C62 210.1 mm to (245.1, 89.1), turned to -90 degrees
- moved PS1 202.6 mm to (254.9, 91.8), turned to -90 degrees
- moved D7 201.7 mm to (253.1, 102.4)
- moved PS4 174.7 mm to (253.8, 136.3), turned to -90 degrees
- moved J5 151.4 mm to (206.2, 101.3)
- moved J1 135.3 mm to (157.7, 119.5)
- moved J4 132.9 mm to (177.8, 101.0)
- moved J3 118.8 mm to (153.3, 106.0), turned to 90 degrees
- moved R4 85.9 mm to (206.8, 65.6), turned to -90 degrees
- moved R18 85.4 mm to (213.8, 65.7), turned to -90 degrees
- moved C1 84.8 mm to (150.7, 95.1)
- moved R9 77.1 mm to (212.2, 65.7), turned to -90 degrees
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
Commit message: placement rough draft
roughly placed all components
Parts:
- added C10: 470pF, Capacitor_SMD:C_0603_1608Metric_Pad1.08x0.95mm_HandSolder, F.Cu at (213.8, 65.7)
- added C13: 470pF, Capacitor_SMD:C_0603_1608Metric_Pad1.08x0.95mm_HandSolder, F.Cu at (165.9, 69.5)
- added C19: 470pF, Capacitor_SMD:C_0603_1608Metric_Pad1.08x0.95mm_HandSolder, F.Cu at (188.5, 69.7)
- added C20: 470pF, Capacitor_SMD:C_0603_1608Metric_Pad1.08x0.95mm_HandSolder, F.Cu at (215.4, 69.9)
- added C7: 470pF, Capacitor_SMD:C_0603_1608Metric_Pad1.08x0.95mm_HandSolder, F.Cu at (164.2, 65.8)
- added C8: 470pF, Capacitor_SMD:C_0603_1608Metric_Pad1.08x0.95mm_HandSolder, F.Cu at (186.9, 65.8)
- C50: moved to B.Cu
- D10, D11, D12, D13: value 5.1-5.7v -> PDZVTFTR5.1B
- moved D13 167.6 mm to (230.4, 100.6), turned to 180 degrees
- moved H4 154.1 mm to (248.3, 44.2)
- moved R44 143.6 mm to (239.9, 100.4), turned to 90 degrees
- moved H3 141.6 mm to (248.0, 110.8)
- moved C66 139.5 mm to (227.8, 88.2), turned to -90 degrees
- moved C67 138.8 mm to (235.8, 99.4)
- moved C65 137.1 mm to (226.0, 88.2), turned to -90 degrees
- moved C3 136.4 mm to (201.2, 95.7)
- moved D1 129.9 mm to (237.1, 101.4)
- moved R77 122.6 mm to (194.0, 51.7), turned to 90 degrees
- moved D3 111.2 mm to (194.0, 55.3), turned to 90 degrees
- moved C2 109.5 mm to (174.9, 95.3)
- moved R2 98.8 mm to (165.8, 51.3), turned to 90 degrees
- moved C50 98.1 mm to (104.8, 70.5), turned to 180 degrees
- moved D2 89.6 mm to (165.8, 54.9), turned to 90 degrees
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Connections:
- D1 pad 1: GND -> HV-

Commit message: some change
Parts:
- added C22: 10nF, Capacitor_SMD:C_0603_1608Metric_Pad1.08x0.95mm_HandSolder, F.Cu at (117.2, 98.3)
- added D13: PDZVTFTR5.1B, Diode_SMD:D_SOD-128, F.Cu at (150.9, 78.9)
- added D14: 300mV 1A, Diode_SMD:D_SOD-123F, F.Cu at (172.4, 101.6)
- added D15: 300mV 1A, Diode_SMD:D_SOD-123F, F.Cu at (214.1, 99.7)
- added D16: 300mV 1A, Diode_SMD:D_SOD-123F, F.Cu at (238.1, 112.5)
- added D17: PDZVTFTR5.1B, Diode_SMD:D_SOD-128, F.Cu at (207.7, 100.0)
- added D18: PDZVTFTR5.1B, Diode_SMD:D_SOD-128, F.Cu at (231.7, 112.8)
- added D19: 300mV 1A, Diode_SMD:D_SOD-123F, F.Cu at (172.4, 105.0)
- added D20: 300mV 1A, Diode_SMD:D_SOD-123F, F.Cu at (214.1, 103.0)
- added D21: 300mV 1A, Diode_SMD:D_SOD-123F, F.Cu at (238.1, 115.8)
- added D22: PDZVTFTR5.1B, Diode_SMD:D_SOD-128, F.Cu at (158.7, 84.0)
- added D23: PDZVTFTR5.1B, Diode_SMD:D_SOD-128, F.Cu at (207.7, 104.0)
- added D24: PDZVTFTR5.1B, Diode_SMD:D_SOD-128, F.Cu at (231.7, 116.9)
- added R17: 0, Resistor_SMD:R_0603_1608Metric_Pad0.98x0.95mm_HandSolder, F.Cu at (237.5, 118.8)
- added R31: 0, Resistor_SMD:R_0603_1608Metric_Pad0.98x0.95mm_HandSolder, F.Cu at (171.8, 110.4)
- added R33: 0, Resistor_SMD:R_0603_1608Metric_Pad0.98x0.95mm_HandSolder, F.Cu at (213.5, 108.4)
- added R34: 0, Resistor_SMD:R_0603_1608Metric_Pad0.98x0.95mm_HandSolder, F.Cu at (237.5, 121.3)
- added R5: 0, Resistor_SMD:R_0603_1608Metric_Pad0.98x0.95mm_HandSolder, F.Cu at (171.8, 107.9)
- added R6: 0, Resistor_SMD:R_0603_1608Metric_Pad0.98x0.95mm_HandSolder, F.Cu at (213.5, 105.9)
- D4, D5, D6: value ~ -> 300mV 1A; footprint Diode_SMD:D_SOD-523 -> Diode_SMD:D_SOD-123F
- R23, R24, R25: footprint LED_SMD:LED_0603_1608Metric_Pad1.05x0.95mm_HandSolder -> Resistor_SMD:R_0603_1608Metric_Pad0.98x0.95mm_HandSolder
- moved C56 43.5 mm to (180.0, 80.5)
- moved C59 43.5 mm to (171.9, 69.2)
- moved C62 43.5 mm to (170.2, 69.2)
- moved D7 43.5 mm to (178.2, 82.5)
- moved PS1 43.5 mm to (180.0, 71.9)
- moved R27 43.5 mm to (181.9, 82.5)
- moved D9 30.0 mm to (253.3, 80.6)
- moved R32 30.0 mm to (256.8, 80.6)
- moved PS3 30.0 mm to (255.4, 70.2)
- moved C58 30.0 mm to (255.0, 78.8)
- moved C61 30.0 mm to (247.2, 67.6)
- moved C64 30.0 mm to (245.5, 67.6)
- moved C38 24.2 mm to (227.8, 64.9)
- moved C46 24.2 mm to (229.3, 80.8)
- moved C55 24.2 mm to (229.3, 79.1)
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Connections:
- D13 pad 1: +5V_HV -> /Phase1/LS_{Gate}
