File: HEI_Logic_Stage/HEI_Logic.kicad_pcb (KiCad board)
At the start: 4 copper layers, 94.6 x 82.8 mm, 165 parts, among them J1 Conn_02x07_Odd_Even, J2 Conn_02x07_Odd_Even, J3 Tag-Connect, J4 430450813_Molex, J7 RJ_{1}, J8 RJ_{2}, SW2 SW_Push, SW3 SW_SPST, U1 CD40109BQNSRQ1, U11 B1203XT-1WR3, U12 5V_Converter_R-78E5.0-0.5, U13 5V_Converter_R-78E5.0-0.5, U14 ADM3058EBRIZ, U16 TLV9051IDBVR, U2 TMH 1212S, U3 TLV9051IDBVR, U4 TLV9051IDBVR, U5 STM32F334C8T6, U6 LM4132-Q1 SOT-2, U7 TLV9051IDBVR, U8 TLV9051IDBVR

Commit message: almost completed new logic layout
Parts:
- added U9: PDS1-S12-S3-M, HEI_Logic:CONV_PDS1-S12-S3-M, F.Cu at (220.0, 114.8)
- C19, C20, C24, C25, JP2, TP18: moved to B.Cu
- J1, J2: footprint Connector_PinHeader_2.54mm:PinHeader_2x07_P2.54mm_Horizontal -> Connector_PinHeader_2.54mm:PinHeader_2x07_P2.54mm_Vertical_SMD; moved to B.Cu
- J4: value 430450813_Molex -> 430451210; footprint Connector_Molex:Molex_Micro-Fit_3.0_43045-0812_2x04_P3.00mm_Vertical -> HEI_Logic:MOLEX_430451210
- R71: value 25k -> 35k
- R72: value 30k -> 40k
- U6: value LM4132-Q1 SOT-2 -> LM4132BMF-3.3
- moved H4 231.1 mm to (247.9, 90.9)
- moved H2 226.3 mm to (247.9, 132.6)
- moved R52 173.7 mm to (199.1, 125.7), turned to 180 degrees
- moved R68 172.2 mm to (196.7, 127.3), turned to 180 degrees
- moved C37 170.5 mm to (196.7, 125.7), turned to 180 degrees
- moved R28 170.0 mm to (204.3, 118.7), turned to 0 degrees
- moved R54 168.7 mm to (199.2, 122.7), turned to 180 degrees
- moved R77 167.8 mm to (201.8, 120.7), turned to 180 degrees
- moved R60 167.6 mm to (194.6, 126.3), turned to 90 degrees
- moved R62 166.4 mm to (204.3, 116.1), turned to 0 degrees
- moved R58 166.4 mm to (194.7, 124.7), turned to 180 degrees
- moved C34 166.3 mm to (201.7, 119.2), turned to 180 degrees
- moved C24 166.1 mm to (213.5, 100.6)
- moved R12 165.6 mm to (214.9, 131.6), turned to 0 degrees
- moved R59 165.5 mm to (192.1, 127.3), turned to 180 degrees
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Connections:
- C17 pad 1: +3V3 -> +5V
- J1 pad 1: GND -> unconnected-(J1-Pin_1-Pad1)
- J1 pad 10: unconnected-(J1-Pin_10-Pad10) -> /HRTIM_D2
- J1 pad 11: /HRTIM_D2 -> unconnected-(J1-Pin_11-Pad11)
- J1 pad 12: unconnected-(J1-Pin_12-Pad12) -> /HRTIM_D1
- J1 pad 13: /HRTIM_D1 -> +12V_MCU
- J1 pad 14: unconnected-(J1-Pin_14-Pad14) -> GND
- J1 pad 2: +12V_MCU -> /HRTIM_B2
- J1 pad 3: /HRTIM_B2 -> unconnected-(J1-Pin_3-Pad3)
- J1 pad 4: unconnected-(J1-Pin_4-Pad4) -> /HRTIM_B1
- J1 pad 5: /HRTIM_B1 -> unconnected-(J1-Pin_5-Pad5)
- J1 pad 6: unconnected-(J1-Pin_6-Pad6) -> /HRTIM_A2
- J1 pad 7: /HRTIM_A2 -> unconnected-(J1-Pin_7-Pad7)
- J1 pad 8: unconnected-(J1-Pin_8-Pad8) -> /HRTIM_A1
- J1 pad 9: /HRTIM_A1 -> unconnected-(J1-Pin_9-Pad9)
- J2 pad 1: GND -> /Control & Motor Interface/DCVsense-
- J2 pad 10: /Control & Motor Interface/DCIsenseRef -> /Control & Motor Interface/PhC_Isense+
- J2 pad 11: /Control & Motor Interface/PhA_IsenseRef -> unconnected-(J2-Pin_11-Pad11)
- J2 pad 12: /Control & Motor Interface/DCVsense+ -> /Control & Motor Interface/PhC_IsenseRef
- J2 pad 13: /Control & Motor Interface/PhA_Isense+ -> +5V
- J2 pad 14: /Control & Motor Interface/DCVsense- -> GND
- J2 pad 2: +5V -> /Control & Motor Interface/PhA_Isense+
- J2 pad 3: /Control & Motor Interface/PhC_IsenseRef -> /Control & Motor Interface/DCVsense+
- J2 pad 4: unconnected-(J2-Pin_4-Pad4) -> /Control & Motor Interface/PhA_IsenseRef
- J2 pad 5: /Control & Motor Interface/PhC_Isense+ -> /Control & Motor Interface/DCIsenseRef
- J2 pad 6: unconnected-(J2-Pin_6-Pad6) -> /Control & Motor Interface/PhB_Isense+
- J2 pad 7: /Control & Motor Interface/PhB_IsenseRef -> /Control & Motor Interface/DCIsense+
- J2 pad 8: /Control & Motor Interface/DCIsense+ -> /Control & Motor Interface/PhB_IsenseRef
- J2 pad 9: /Control & Motor Interface/PhB_Isense+ -> unconnected-(J2-Pin_9-Pad9)
- J4 pad 3: Net-(J4-Pad3) -> GND
- J4 pad 4: Net-(J4-Pad4) -> /Control & Motor Interface/TIN1_r
- J4 pad 5: GND -> /Control & Motor Interface/TIN2_r
- J4 pad 6: Net-(J4-Pad6) -> /Control & Motor Interface/TIN3_r
- J4 pad 7: Net-(J4-Pad7) -> GND
- R14 pad 2: Net-(J4-Pad4) -> /Control & Motor Interface/TIN2_r
- R2 pad 2: Net-(J4-Pad8) -> /Control & Motor Interface/TIN3_r
- R22 pad 1: Net-(J4-Pad6) -> Net-(J4-Pad8)
- R23 pad 2: Net-(J4-Pad3) -> /Control & Motor Interface/TIN1_r
- R24 pad 1: Net-(J4-Pad7) -> Net-(J4-Pad9)
- R33 pad 1: Net-(J4-Pad8) -> /Control & Motor Interface/TIN3_r
- R34 pad 1: Net-(J4-Pad3) -> /Control & Motor Interface/TIN1_r
- R35 pad 1: Net-(J4-Pad4) -> /Control & Motor Interface/TIN2_r
- TP20 pad 1: /HRTIM_D1 -> /HRTIM_B2
- TP21 pad 1: /HRTIM_D2 -> /HRTIM_B1
- TP24 pad 1: /HRTIM_A1 -> /HRTIM_A2
- TP25 pad 1: /HRTIM_A2 -> /HRTIM_A1
- TP26 pad 1: /HRTIM_B1 -> /HRTIM_D2
- TP27 pad 1: /HRTIM_B2 -> /HRTIM_D1
- U6 pad 3: +3V3 -> +5V
- U6 pad 4: +3V3 -> +5V
Routing:
- net /Vref: track 0.00 -> 98.0 mm, vias 0 -> 10
- net /~{RST}: track 0.00 -> 48.2 mm, vias 0 -> 2
- net /Control & Motor Interface/DCVsense-: track 17.4 -> 59.6 mm, vias 0 -> 2
- net /LED3: track 41.9 -> 1.22 mm, vias 2 -> 1
- net /HallIN3_3v3: track 0.00 -> 38.3 mm, vias 0 -> 2
- net /LED2: track 39.1 -> 1.22 mm, vias 2 -> 1
- net /HallIN2_3v3: track 0.00 -> 36.7 mm, vias 0 -> 2
- net /Control & Motor Interface/TIN1_r: track 0.00 -> 36.1 mm
- net /Control & Motor Interface/TIN3_r: track 0.00 -> 35.4 mm
- net /HallIN1_3v3: track 0.00 -> 35.3 mm, vias 0 -> 2
- net /Control & Motor Interface/DCVsense+: track 25.8 -> 60.9 mm, vias 0 -> 2
- net /LED1: track 36.8 -> 1.73 mm, vias 2 -> 1
- net Net-(J4-Pad9): track 0.00 -> 33.4 mm
- net /Control & Motor Interface/TIN2_r: track 0.00 -> 30.2 mm
- net /SWDCLK: track 19.2 -> 49.3 mm
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- removed copper zone on F.Cu, net +12V_MCU
- removed copper zone on In2.Cu, net +12V_MCU
Other:
- board size 94.6 x 82.8 mm -> 95.8 x 46.7 mm
- board text added: "12V_MCU"
- board text added: "HEI Logic"
- board text added: "rev1 sept. 2024"
- board text removed: "12V MCU"
- board text removed: "ALIGNMENT FIX!"
- board text removed: "High Efficiency Inverter - Logic Stage"

Commit message: main portion of logic drc done
Parts:
- C19, C20, C24, C25, JP2, TP18: moved to F.Cu
- moved R27 172.4 mm to (1.68, -2.03)
- moved TP18 33.5 mm to (170.9, 91.4), turned to 0 degrees
- moved TP19 16.9 mm to (242.6, 91.4), turned to 90 degrees
- moved C19 16.7 mm to (206.0, 98.8), turned to 90 degrees
- moved JP2 14.4 mm to (204.5, 94.7), turned to -90 degrees
- moved C20 13.2 mm to (231.1, 91.5)
- moved C24 12.4 mm to (206.0, 90.7), turned to -90 degrees
- moved TP2 12.1 mm to (238.5, 91.4), turned to 90 degrees
- moved TP1 7.28 mm to (234.4, 91.4), turned to 90 degrees
- moved C25 6.25 mm to (226.8, 102.6), turned to 0 degrees
- moved TP15 4.23 mm to (205.4, 109.7)
- moved TP16 4.23 mm to (205.5, 112.8)
- moved D5 2.80 mm to (211.0, 131.3)
- moved R13 2.80 mm to (214.9, 131.3)
- moved D4 2.29 mm to (210.9, 133.9)
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Connections:
- U5 pad 22: unconnected-(U5-PB11-Pad22) -> /LED3
- U5 pad 25: unconnected-(U5-PB12-Pad25) -> /LED2
- U5 pad 26: unconnected-(U5-PB13-Pad26) -> /LED1
- U5 pad 39: /LED1 -> unconnected-(U5-PB3-Pad39)
- U5 pad 40: /LED2 -> unconnected-(U5-PB4-Pad40)
- U5 pad 41: /LED3 -> unconnected-(U5-PB5-Pad41)
Routing:
- net GND: track 17.9 -> 153.3 mm, vias 12 -> 52
- net +5V: track 4.58 -> 81.1 mm, vias 0 -> 6
- net /LED2: track 1.22 -> 77.3 mm, vias 1 -> 2
- net /LED1: track 1.73 -> 76.4 mm, vias 1 -> 2
- net /LED3: track 1.22 -> 73.6 mm, vias 1 -> 2
- net +12V_MCU: track 0.00 -> 62.3 mm
- net +5V_CAN: track 0.00 -> 48.3 mm, vias 0 -> 1
- net GND_LV: track 0.00 -> 38.3 mm, vias 0 -> 6
- net +3V3: track 9.75 -> 33.2 mm, vias 8 -> 16
- net /Control & Motor Interface/PhA_Isense+: track 33.4 -> 22.0 mm
- net V_Hall: track 0.00 -> 9.14 mm, vias 0 -> 6
- net /Control & Motor Interface/PhA_IsenseRef: track 36.0 -> 27.9 mm
- net +12V_LV: track 0.00 -> 6.38 mm, vias 0 -> 3
- net /Vref: track 98.0 -> 102.6 mm
- net /Control & Motor Interface/DCVsense+: track 60.9 -> 58.6 mm
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- added copper zone on F.Cu, net V_Hall
- added copper zone on In2.Cu, net V_Hall
Other:
- board text added: "12V"
- board text added: "12V | GND_LV | 5V"
- board text added: "5V"
- board text added: "to HEI Power"
- board text removed: "12V_MCU"

Commit message: final tweaks to logic, silkscreen not done
Parts:
- removed SW2: SW_Push, GTSR_KiCAD_Footprints:KMR223GLFG
- removed U11: B1203XT-1WR3, GTSR_KiCAD_Footprints:B_XT-1WR3_MNS-M
- added FB1: ~, Resistor_SMD:R_0805_2012Metric, B.Cu at (211.0, 97.6)
- added FB2: ~, Resistor_SMD:R_0805_2012Metric, B.Cu at (184.2, 95.1)
- added SW1: KMR223GLFG, HEI_Logic:KMR223GLFG, F.Cu at (157.2, 110.7)
- R27: moved to B.Cu
- moved R27 211.2 mm to (177.8, 114.6), turned to 90 degrees
- moved TP11 24.4 mm to (167.9, 91.4)
- moved H1 0.56 mm to (157.5, 133.1)
- moved H4 0.25 mm to (247.9, 90.7)
Connections:
- J1 pad 1: unconnected-(J1-Pin_1-Pad1) -> GND
- J1 pad 11: unconnected-(J1-Pin_11-Pad11) -> GND
- J1 pad 13: +12V_MCU -> Net-(J1-Pin_13)
- J1 pad 3: unconnected-(J1-Pin_3-Pad3) -> GND
- J1 pad 5: unconnected-(J1-Pin_5-Pad5) -> GND
- J1 pad 7: unconnected-(J1-Pin_7-Pad7) -> GND
- J1 pad 9: unconnected-(J1-Pin_9-Pad9) -> GND
- J2 pad 11: unconnected-(J2-Pin_11-Pad11) -> GND
- J2 pad 13: +5V -> Net-(J2-Pin_13)
- J2 pad 9: unconnected-(J2-Pin_9-Pad9) -> GND
- R27 pad 2: /Unused -> Net-(U5-PH3-BOOT0)
- U5 pad 3: /Unused -> unconnected-(U5-PC14-OSC32_IN-Pad3)
- U5 pad 4: /Unused -> unconnected-(U5-PC15-OSC32_OUT-Pad4)
- U5 pad 44: /Unused -> Net-(U5-PH3-BOOT0)
- U5 pad 5: /Unused -> unconnected-(U5-PH0-OSC_IN-Pad5)
- U5 pad 6: /Unused -> unconnected-(U5-PH1-OSC_OUT-Pad6)
Routing:
- net Net-(U5-PH3-BOOT0): track 0.00 -> 6.86 mm, vias 0 -> 1
- net GND: track 153.3 -> 160.0 mm, vias 52 -> 56
- net /Vref: track 102.6 -> 108.1 mm
- net Net-(J2-Pin_13): track 0.00 -> 5.12 mm
- net /Power & CAN/CANL: track 39.9 -> 44.4 mm
- net Net-(J1-Pin_13): track 0.00 -> 3.83 mm
- net +12V_MCU: track 62.3 -> 58.8 mm
- net +5V: track 81.1 -> 83.6 mm
- net /Control & Motor Interface/DCIsense+: track 49.6 -> 51.8 mm
- net /Control & Motor Interface/DCVsense-: track 58.7 -> 59.8 mm
- net /Control & Motor Interface/PhA_Isense+: track 22.0 -> 23.1 mm
- net /Power & CAN/CANH: track 55.2 -> 56.1 mm
- net GND_LV: track 38.3 -> 39.1 mm, vias 6 -> 7
- net /Control & Motor Interface/DCVsense+: track 58.6 -> 59.2 mm
- net /UART_RX: track 31.1 -> 31.7 mm
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Other:
- board text added: "12V | VHall | 5V"
- board text added: "RST"
- board text added: "Vref"
